Commit message: xacro error

File: urdf/macros.xacro (robot description, xacro)
@@ -1,5 +1,5 @@
 <?xml version="1.0"?>
-<robot>
-  <macro name="cylinder_inertial" params="name m r h">
+<robot xmlns:xacro="http://www.ros.org/wiki/xacro">
+  <xacro:macro name="cylinder_inertial" params="name m r h">
     <inertial name="${name}_inertial">
       <mass value="${m}"/>
@@ -8,6 +8,6 @@
         izz="${m*r*r/2}"/>
     </inertial>
-  </macro>
-  <macro name="box_inertial" params="name m x y z">
+  </xacro:macro>
+  <xacro:macro name="box_inertial" params="name m x y z">
     <inertial name="${name}_inertial">
       <mass value="${m}"/>
@@ -16,6 +16,6 @@
         izz="${m*(x*x+z*z)/12}"/>
     </inertial>
-  </macro>
-  <macro name="sphere_inertial" params="name m r">
+  </xacro:macro>
+  <xacro:macro name="sphere_inertial" params="name m r">
     <inertial name="${name}_inertial">
       <mass value="${m}"/>
@@ -24,4 +24,4 @@
         izz="${2*m*r*r/5}"/>
     </inertial>
-  </macro>
+  </xacro:macro>
 </robot>
