Commit message: world update and trying to simulate D435i

File: urdf/robot_leader.xacro (robot description, xacro)
@@ -16,4 +16,5 @@
   <xacro:include filename="$(find smartcarts)/urdf/macros.xacro"/>
   <xacro:include filename="$(find smartcarts)/urdf/materials.xacro"/>
+  <xacro:include filename="$(find smartcarts)/urdf/realsense_d435.urdf.xacro" />
   <link name='chassis'>
     <xacro:box_inertial name="chassis" m="${chassis_mass}" x="${chassis_length}" y="${chassis_width}" z="${chassis_height}"/>
@@ -110,5 +111,5 @@
     </visual>
   </link>
- <!--  <link name='camera_link'>
+ <link name='camera_link'>
     <xacro:box_inertial name="camera_link" m="${camera_mass}" x="${camera_width}" y="${camera_length}" z="${camera_height}"/>
     <collision name='camera_link_collision'>
@@ -123,5 +124,5 @@
       </geometry>
     </visual>
-  </link> -->
+  </link>
   <link name="imu_link">
     <inertial>
@@ -143,4 +144,9 @@
     </collision>
   </link>
+  <sensor_d435 parent="camera_link">
+    <topic>__default_topic__</topic>
+    <topicName>realsense_camera</topicName>
+    <origin xyz="0.0 0.2 0" rpy="0 0 0"/>
+  </sensor_d435>
   <joint name="ball_joint" type="continuous">
     <parent link="chassis"/>
@@ -176,9 +182,9 @@
     <axis xyz="0 1 0"/>
   </joint>
-  <!-- <joint name="camera_joint" type="fixed">
+  <joint name="camera_joint" type="fixed">
     <parent link="chassis"/>
     <child link="camera_link"/>
     <origin xyz="${chassis_length/2} 0 ${chassis_height/2+camera_height/2}"/>
-  </joint> -->
+  </joint>
   <joint name="imu_link" type="fixed">
     <axis xyz="1 0 0"/> <!-- 0 1 0 -->
@@ -250,6 +256,6 @@
     </plugin>
   </gazebo>
-<!--   <gazebo reference="camera_link">
-    <sensor type="camera" name="camera1">
+  <gazebo reference="camera_link">
+    <sensor type="camera" name="realsense_d435">
       <update_rate>30.0</update_rate>
       <camera name="head">
@@ -273,5 +279,5 @@
         <alwaysOn>true</alwaysOn>
         <updateRate>0.0</updateRate>
-        <cameraName>camera1</cameraName>
+        <cameraName>realsense_d435</cameraName>
         <imageTopicName>image_raw</imageTopicName>
         <cameraInfoTopicName>camera_info</cameraInfoTopicName>
@@ -285,5 +291,5 @@
       </plugin>
     </sensor>
-  </gazebo> -->
+  </gazebo>
 <!--
   <xacro:property name="camera_name" value="camera1"/>

Commit message: testing simulation

File: urdf/robot_leader.xacro (robot description, xacro)
@@ -16,5 +16,4 @@
   <xacro:include filename="$(find smartcarts)/urdf/macros.xacro"/>
   <xacro:include filename="$(find smartcarts)/urdf/materials.xacro"/>
-  <xacro:include filename="$(find smartcarts)/urdf/realsense_d435.urdf.xacro" />
   <link name='chassis'>
     <xacro:box_inertial name="chassis" m="${chassis_mass}" x="${chassis_length}" y="${chassis_width}" z="${chassis_height}"/>
@@ -111,5 +110,5 @@
     </visual>
   </link>
- <link name='camera_link'>
+ <!-- <link name='camera_link'>
     <xacro:box_inertial name="camera_link" m="${camera_mass}" x="${camera_width}" y="${camera_length}" z="${camera_height}"/>
     <collision name='camera_link_collision'>
@@ -124,5 +123,5 @@
       </geometry>
     </visual>
-  </link>
+  </link>  -->
   <link name="imu_link">
     <inertial>
@@ -144,9 +143,9 @@
     </collision>
   </link>
-  <sensor_d435 parent="camera_link">
+  <!-- <sensor_d435 parent="camera_link">
     <topic>__default_topic__</topic>
     <topicName>realsense_camera</topicName>
     <origin xyz="0.0 0.2 0" rpy="0 0 0"/>
-  </sensor_d435>
+  </sensor_d435> -->
   <joint name="ball_joint" type="continuous">
     <parent link="chassis"/>
@@ -256,5 +255,5 @@
     </plugin>
   </gazebo>
-  <gazebo reference="camera_link">
+  <!-- <gazebo reference="camera_link">
     <sensor type="camera" name="realsense_d435">
       <update_rate>30.0</update_rate>
@@ -291,5 +290,5 @@
       </plugin>
     </sensor>
-  </gazebo>
+  </gazebo> -->
 <!--
   <xacro:property name="camera_name" value="camera1"/>
